File: kicad/Amperometro-con-soglia-cablaggio.kicad_sch (KiCad schematic)
At the start: 13 parts, among them J1 IDC_13X2, J10 MAMMUT, J2 Conn_01x03_Pin, J3 Conn_01x03_Pin, J4 Conn_01x04_Pin, J5 Conn_01x03_Pin, J6 Barrel_Jack, J7 banana nera, J8 banana rossa, J9 Conn_01x04_Pin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

Commit message: schema con sim
Parts:
- added SW2: SW_DPST_x2, symbol Switch:SW_DPST_x2
- added U1: L7812, symbol Regulator_Linear:L7812
Connections:
- net +12: now also U1.3 (OUT); no longer J6.1
- net D2: now also SW2.2 (B); no longer BZ1.2 (-)
- net GND: now also U1.2 (GND)
- new net: BZ1.2 (-), SW2.1 (A)
- new net +24V: J6.1, U1.1 (IN)
Other:
- note added: "relay allarme"
- moved on the sheet: BZ1, J1, J10, J2, J3, J4, J5, J6, J7, J8, J9, RV1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

Commit message: schemi definitivi
Parts:
- removed J4: Conn_01x04_Pin, symbol Connector:Conn_01x04_Pin
- removed U1: L7812, symbol Regulator_Linear:L7812
- added J11: DE9_Pins, symbol Connector:DE9_Pins
- added J12: DE9_Socket, symbol Connector:DE9_Socket
- added J13: Conn_01x04_Pin, symbol Connector:Conn_01x04_Pin
- added SW3: SW_DPST_x2, symbol Switch:SW_DPST_x2
Connections:
- net +12: now also J6.1, SW3.1 (A)
- net +24V: no longer J6.1
- net +5: now also J13.2 (Pin_2)
- net GND: now also J13.1 (Pin_1)
- net SCK: now also J13.3 (Pin_3)
- net SDA: now also J13.4 (Pin_4)
Other:
- note added: "BIA-RXSIM"
- note added: "GIA-TXSIM"
- note added: "ROS-ARA-VIO-BRU"
- note added: "RX"
- note added: "TX"
- note added: "VER-BLU-NER-SCH"
- note added: "XL6009 Boost Buck DC-DC"
- note added: "sensore LEM CTSR 1P"
- note added: "sim800"
- note removed: "sensore LEM"
- moved on the sheet: BZ1, J1, J10, J2, J3, J5, J6, J7, J8, J9, RV1, SW1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
